File: Bad Apple/pwr_sys.kicad_sch (KiCad schematic)
At the start: 0 parts

Commit message: feat(pcb): more hierarchy
Other:
- company: (none) -> Mixed Engineering Group 3 | STEM 12-Altruism / AY 2526 | CIT-U SHS
- title: (none) -> Autonomous  Courier Robot "Bad Apple"
Changed lines of the file:
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@@
 	(generator_version "9.0")
 	(paper "A4")
+	(title_block
+		(title "Autonomous  Courier Robot \"Bad Apple\"")
+		(date "2025-08-28")
+		(rev "1")
+		(company "Mixed Engineering Group 3 | STEM 12-Altruism / AY 2526 | CIT-U SHS")
+		(comment 4 "5V ~1A power supply for the raspberry pi and the hat's peripherals")
+	)
 )
